File: scrabblepad.sch (KiCad schematic (older format))
At the start: 475 parts, among them P1 pad, P10 pad, P11 pad, P12 pad, P13 pad, P14 pad, P15 pad, P16 pad, P2 pad, P3 pad, P4 pad, P5 pad, P6 pad, P7 pad, P8 pad, P9 pad, T1 TRRS, U1 Teensy++2.0, q1 quadpad, q2 quadpad

Commit message: cleanup, library management
Parts:
- removed q1, q2: quadpad, donutbrary:quadpad, symbol donutbrary:QuadPad
- added Q1, Q2: Quad_Pad, symbol donutbrary:Quad_Pad
- RGB1: renamed from rgb1; value rgb_pad -> RGB_Pad
- SD1: value teensy_sd -> Teensy_SD; footprint donutbrary:teensy_sd -> (none)
Connections:
- wire segments 434 -> 440
Other:
- moved on the sheet: P1, P10, P11, P12, P13, P14, P15, P16, P2, P3, P4, P5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

Commit message: update/cleanup
Parts:
- D1, D10, D100, D101, D102, D103, D104, D105, D106, D107, D108, D109, D11, D110, D111, D112, D113, D114, D115, D116, D117, D118, D119, D12, D120, D121, D122, D123, D124, D125, D126, D127, D128, D129, D13, D130, D131, D132, D133, D134, D135, D136, D137, D138, D139, D14, D140, D141, D142, D143, D144, D145, D146, D147, D148, D149, D15, D150, D151, D152, D153, D154, D155, D156, D157, D158, D159, D16, D160, D161, D162, D163, D164, D165, D166, D167, D168, D169, D17, D170, D171, D172, D173, D174, D175, D176, D177, D178, D179, D18, D180, D181, D182, D183, D184, D185, D186, D187, D188, D189, D19, D190, D191, D192, D193, D194, D195, D196, D197, D198, D199, D2, D20, D200, D201, D202, D203, D204, D205, D206, D207, D208, D209, D21, D210, D211, D212, D213, D214, D215, D216, D217, D218, D219, D22, D220, D221, D222, D223, D224, D225, D23, D24, D25, D26, D27, D28, D29, D3, D30, D31, D32, D33, D34, D35, D36, D37, D38, D39, D4, D40, D41, D42, D43, D44, D45, D46, D47, D48, D49, D5, D50, D51, D52, D53, D54, D55, D56, D57, D58, D59, D6, D60, D61, D62, D63, D64, D65, D66, D67, D68, D69, D7, D70, D71, D72, D73, D74, D75, D76, D77, D78, D79, D8, D80, D81, D82, D83, D84, D85, D86, D87, D88, D89, D9, D90, D91, D92, D93, D94, D95, D96, D97, D98, D99: symbol donutbrary:D12 -> donutbrary:D21
Connections:
- net Row0: now also D1.1 (C), D10.1 (C), D11.1 (C), D12.1 (C), D13.1 (C), D14.1 (C), D15.1 (C), D2.1 (C), D3.1 (C), D4.1 (C), D5.1 (C), D6.1 (C), D7.1 (C), D8.1 (C), D9.1 (C); no longer D1.2 (A), D10.2 (A), D11.2 (A), D12.2 (A), D13.2 (A), D14.2 (A), D15.2 (A), D2.2 (A), D3.2 (A), D4.2 (A), D5.2 (A), D6.2 (A), D7.2 (A), D8.2 (A), D9.2 (A)
- net Row1: now also D16.1 (C), D17.1 (C), D18.1 (C), D19.1 (C), D20.1 (C), D21.1 (C), D22.1 (C), D23.1 (C), D24.1 (C), D25.1 (C), D26.1 (C), D27.1 (C), D28.1 (C), D29.1 (C), D30.1 (C); no longer D16.2 (A), D17.2 (A), D18.2 (A), D19.2 (A), D20.2 (A), D21.2 (A), D22.2 (A), D23.2 (A), D24.2 (A), D25.2 (A), D26.2 (A), D27.2 (A), D28.2 (A), D29.2 (A), D30.2 (A)
- net Row10: now also D151.1 (C), D152.1 (C), D153.1 (C), D154.1 (C), D155.1 (C), D156.1 (C), D157.1 (C), D158.1 (C), D159.1 (C), D160.1 (C), D161.1 (C), D162.1 (C), D163.1 (C), D164.1 (C), D165.1 (C); no longer D151.2 (A), D152.2 (A), D153.2 (A), D154.2 (A), D155.2 (A), D156.2 (A), D157.2 (A), D158.2 (A), D159.2 (A), D160.2 (A), D161.2 (A), D162.2 (A), D163.2 (A), D164.2 (A), D165.2 (A)
- net Row11: now also D166.1 (C), D167.1 (C), D168.1 (C), D169.1 (C), D170.1 (C), D171.1 (C), D172.1 (C), D173.1 (C), D174.1 (C), D175.1 (C), D176.1 (C), D177.1 (C), D178.1 (C), D179.1 (C), D180.1 (C); no longer D166.2 (A), D167.2 (A), D168.2 (A), D169.2 (A), D170.2 (A), D171.2 (A), D172.2 (A), D173.2 (A), D174.2 (A), D175.2 (A), D176.2 (A), D177.2 (A), D178.2 (A), D179.2 (A), D180.2 (A)
- net Row12: now also D181.1 (C), D182.1 (C), D183.1 (C), D184.1 (C), D185.1 (C), D186.1 (C), D187.1 (C), D188.1 (C), D189.1 (C), D190.1 (C), D191.1 (C), D192.1 (C), D193.1 (C), D194.1 (C), D195.1 (C); no longer D181.2 (A), D182.2 (A), D183.2 (A), D184.2 (A), D185.2 (A), D186.2 (A), D187.2 (A), D188.2 (A), D189.2 (A), D190.2 (A), D191.2 (A), D192.2 (A), D193.2 (A), D194.2 (A), D195.2 (A)
- net Row13: now also D196.1 (C), D197.1 (C), D198.1 (C), D199.1 (C), D200.1 (C), D201.1 (C), D202.1 (C), D203.1 (C), D204.1 (C), D205.1 (C), D206.1 (C), D207.1 (C), D208.1 (C), D209.1 (C), D210.1 (C); no longer D196.2 (A), D197.2 (A), D198.2 (A), D199.2 (A), D200.2 (A), D201.2 (A), D202.2 (A), D203.2 (A), D204.2 (A), D205.2 (A), D206.2 (A), D207.2 (A), D208.2 (A), D209.2 (A), D210.2 (A)
- net Row14: now also D211.1 (C), D212.1 (C), D213.1 (C), D214.1 (C), D215.1 (C), D216.1 (C), D217.1 (C), D218.1 (C), D219.1 (C), D220.1 (C), D221.1 (C), D222.1 (C), D223.1 (C), D224.1 (C), D225.1 (C); no longer D211.2 (A), D212.2 (A), D213.2 (A), D214.2 (A), D215.2 (A), D216.2 (A), D217.2 (A), D218.2 (A), D219.2 (A), D220.2 (A), D221.2 (A), D222.2 (A), D223.2 (A), D224.2 (A), D225.2 (A)
- net Row2: now also D31.1 (C), D32.1 (C), D33.1 (C), D34.1 (C), D35.1 (C), D36.1 (C), D37.1 (C), D38.1 (C), D39.1 (C), D40.1 (C), D41.1 (C), D42.1 (C), D43.1 (C), D44.1 (C), D45.1 (C); no longer D31.2 (A), D32.2 (A), D33.2 (A), D34.2 (A), D35.2 (A), D36.2 (A), D37.2 (A), D38.2 (A), D39.2 (A), D40.2 (A), D41.2 (A), D42.2 (A), D43.2 (A), D44.2 (A), D45.2 (A)
- net Row3: now also D46.1 (C), D47.1 (C), D48.1 (C), D49.1 (C), D50.1 (C), D51.1 (C), D52.1 (C), D53.1 (C), D54.1 (C), D55.1 (C), D56.1 (C), D57.1 (C), D58.1 (C), D59.1 (C), D60.1 (C); no longer D46.2 (A), D47.2 (A), D48.2 (A), D49.2 (A), D50.2 (A), D51.2 (A), D52.2 (A), D53.2 (A), D54.2 (A), D55.2 (A), D56.2 (A), D57.2 (A), D58.2 (A), D59.2 (A), D60.2 (A)
- net Row4: now also D61.1 (C), D62.1 (C), D63.1 (C), D64.1 (C), D65.1 (C), D66.1 (C), D67.1 (C), D68.1 (C), D69.1 (C), D70.1 (C), D71.1 (C), D72.1 (C), D73.1 (C), D74.1 (C), D75.1 (C); no longer D61.2 (A), D62.2 (A), D63.2 (A), D64.2 (A), D65.2 (A), D66.2 (A), D67.2 (A), D68.2 (A), D69.2 (A), D70.2 (A), D71.2 (A), D72.2 (A), D73.2 (A), D74.2 (A), D75.2 (A)
- net Row5: now also D76.1 (C), D77.1 (C), D78.1 (C), D79.1 (C), D80.1 (C), D81.1 (C), D82.1 (C), D83.1 (C), D84.1 (C), D85.1 (C), D86.1 (C), D87.1 (C), D88.1 (C), D89.1 (C), D90.1 (C); no longer D76.2 (A), D77.2 (A), D78.2 (A), D79.2 (A), D80.2 (A), D81.2 (A), D82.2 (A), D83.2 (A), D84.2 (A), D85.2 (A), D86.2 (A), D87.2 (A), D88.2 (A), D89.2 (A), D90.2 (A)
- net Row6: now also D100.1 (C), D101.1 (C), D102.1 (C), D103.1 (C), D104.1 (C), D105.1 (C), D91.1 (C), D92.1 (C), D93.1 (C), D94.1 (C), D95.1 (C), D96.1 (C), D97.1 (C), D98.1 (C), D99.1 (C); no longer D100.2 (A), D101.2 (A), D102.2 (A), D103.2 (A), D104.2 (A), D105.2 (A), D91.2 (A), D92.2 (A), D93.2 (A), D94.2 (A), D95.2 (A), D96.2 (A), D97.2 (A), D98.2 (A), D99.2 (A)
- net Row7: now also D106.1 (C), D107.1 (C), D108.1 (C), D109.1 (C), D110.1 (C), D111.1 (C), D112.1 (C), D113.1 (C), D114.1 (C), D115.1 (C), D116.1 (C), D117.1 (C), D118.1 (C), D119.1 (C), D120.1 (C); no longer D106.2 (A), D107.2 (A), D108.2 (A), D109.2 (A), D110.2 (A), D111.2 (A), D112.2 (A), D113.2 (A), D114.2 (A), D115.2 (A), D116.2 (A), D117.2 (A), D118.2 (A), D119.2 (A), D120.2 (A)
- net Row8: now also D121.1 (C), D122.1 (C), D123.1 (C), D124.1 (C), D125.1 (C), D126.1 (C), D127.1 (C), D128.1 (C), D129.1 (C), D130.1 (C), D131.1 (C), D132.1 (C), D133.1 (C), D134.1 (C), D135.1 (C); no longer D121.2 (A), D122.2 (A), D123.2 (A), D124.2 (A), D125.2 (A), D126.2 (A), D127.2 (A), D128.2 (A), D129.2 (A), D130.2 (A), D131.2 (A), D132.2 (A), D133.2 (A), D134.2 (A), D135.2 (A)
- net Row9: now also D136.1 (C), D137.1 (C), D138.1 (C), D139.1 (C), D140.1 (C), D141.1 (C), D142.1 (C), D143.1 (C), D144.1 (C), D145.1 (C), D146.1 (C), D147.1 (C), D148.1 (C), D149.1 (C), D150.1 (C); no longer D136.2 (A), D137.2 (A), D138.2 (A), D139.2 (A), D140.2 (A), D141.2 (A), D142.2 (A), D143.2 (A), D144.2 (A), D145.2 (A), D146.2 (A), D147.2 (A), D148.2 (A), D149.2 (A), D150.2 (A)
- net at SW_1.2: now also D1.2 (A); no longer D1.1 (C)
- net at SW_2.2: now also D2.2 (A); no longer D2.1 (C)
- net at SW_3.2: now also D3.2 (A); no longer D3.1 (C)
- net at SW_4.2: now also D4.2 (A); no longer D4.1 (C)
- net at SW_5.2: now also D5.2 (A); no longer D5.1 (C)
- net at SW_6.2: now also D6.2 (A); no longer D6.1 (C)
- net at SW_7.2: now also D7.2 (A); no longer D7.1 (C)
- net at SW_8.2: now also D8.2 (A); no longer D8.1 (C)
- net at SW_9.1: now also D9.2 (A); no longer D9.1 (C)
- net at SW_10.2: now also D10.2 (A); no longer D10.1 (C)
- net at SW_11.2: now also D11.2 (A); no longer D11.1 (C)
- net at SW_12.2: now also D12.2 (A); no longer D12.1 (C)
- net at SW_13.2: now also D13.2 (A); no longer D13.1 (C)
- net at SW_14.2: now also D14.2 (A); no longer D14.1 (C)
- net at SW_15.2: now also D15.2 (A); no longer D15.1 (C)
- net at SW_16.2: now also D16.2 (A); no longer D16.1 (C)
- net at SW_17.2: now also D17.2 (A); no longer D17.1 (C)
- net at SW_18.2: now also D18.2 (A); no longer D18.1 (C)
- net at SW_19.2: now also D19.2 (A); no longer D19.1 (C)
- net at SW_20.2: now also D20.2 (A); no longer D20.1 (C)
- net at SW_21.2: now also D21.2 (A); no longer D21.1 (C)
- net at SW_22.2: now also D22.2 (A); no longer D22.1 (C)
- net at SW_23.2: now also D23.2 (A); no longer D23.1 (C)
- net at SW_24.2: now also D24.2 (A); no longer D24.1 (C)
- net at SW_25.2: now also D25.2 (A); no longer D25.1 (C)
- net at SW_26.2: now also D26.2 (A); no longer D26.1 (C)
- net at SW_27.2: now also D27.2 (A); no longer D27.1 (C)
- net at SW_28.2: now also D28.2 (A); no longer D28.1 (C)
- net at SW_29.2: now also D29.2 (A); no longer D29.1 (C)
- net at SW_30.2: now also D30.2 (A); no longer D30.1 (C)
- net at SW_31.2: now also D31.2 (A); no longer D31.1 (C)
- net at SW_32.2: now also D32.2 (A); no longer D32.1 (C)
- net at SW_33.2: now also D33.2 (A); no longer D33.1 (C)
- net at SW_34.2: now also D34.2 (A); no longer D34.1 (C)
- net at SW_35.2: now also D35.2 (A); no longer D35.1 (C)
- net at SW_36.2: now also D36.2 (A); no longer D36.1 (C)
- net at SW_37.2: now also D37.2 (A); no longer D37.1 (C)
- net at SW_38.2: now also D38.2 (A); no longer D38.1 (C)
- net at SW_39.1: now also D39.2 (A); no longer D39.1 (C)
- net at SW_40.2: now also D40.2 (A); no longer D40.1 (C)
- net at SW_41.2: now also D41.2 (A); no longer D41.1 (C)
- net at SW_42.2: now also D42.2 (A); no longer D42.1 (C)
- net at SW_43.2: now also D43.2 (A); no longer D43.1 (C)
- net at SW_44.2: now also D44.2 (A); no longer D44.1 (C)
- net at SW_45.2: now also D45.2 (A); no longer D45.1 (C)
- net at SW_46.2: now also D46.2 (A); no longer D46.1 (C)
- net at SW_47.2: now also D47.2 (A); no longer D47.1 (C)
- net at SW_48.2: now also D48.2 (A); no longer D48.1 (C)
- net at SW_49.2: now also D49.2 (A); no longer D49.1 (C)
- net at SW_50.2: now also D50.2 (A); no longer D50.1 (C)
- net at SW_51.2: now also D51.2 (A); no longer D51.1 (C)
- net at SW_52.2: now also D52.2 (A); no longer D52.1 (C)
- net at SW_53.2: now also D53.2 (A); no longer D53.1 (C)
- net at SW_54.2: now also D54.2 (A); no longer D54.1 (C)
- net at SW_55.2: now also D55.2 (A); no longer D55.1 (C)
- net at SW_56.2: now also D56.2 (A); no longer D56.1 (C)
- net at SW_57.2: now also D57.2 (A); no longer D57.1 (C)
- net at SW_58.2: now also D58.2 (A); no longer D58.1 (C)
- net at SW_59.2: now also D59.2 (A); no longer D59.1 (C)
- net at SW_60.2: now also D60.2 (A); no longer D60.1 (C)
- net at SW_61.2: now also D61.2 (A); no longer D61.1 (C)
- net at SW_62.2: now also D62.2 (A); no longer D62.1 (C)
- net at SW_63.2: now also D63.2 (A); no longer D63.1 (C)
- net at SW_64.2: now also D64.2 (A); no longer D64.1 (C)
- net at SW_65.2: now also D65.2 (A); no longer D65.1 (C)
- net at SW_66.2: now also D66.2 (A); no longer D66.1 (C)
- net at SW_67.2: now also D67.2 (A); no longer D67.1 (C)
- net at SW_68.2: now also D68.2 (A); no longer D68.1 (C)
- net at SW_69.2: now also D69.2 (A); no longer D69.1 (C)
- net at SW_70.2: now also D70.2 (A); no longer D70.1 (C)
- net at SW_71.2: now also D71.2 (A); no longer D71.1 (C)
- net at SW_72.2: now also D72.2 (A); no longer D72.1 (C)
- net at SW_73.2: now also D73.2 (A); no longer D73.1 (C)
- net at SW_74.2: now also D74.2 (A); no longer D74.1 (C)
- net at SW_75.2: now also D75.2 (A); no longer D75.1 (C)
- net at SW_76.2: now also D76.2 (A); no longer D76.1 (C)
- net at SW_77.2: now also D77.2 (A); no longer D77.1 (C)
- net at SW_78.2: now also D78.2 (A); no longer D78.1 (C)
- net at SW_79.2: now also D79.2 (A); no longer D79.1 (C)
- net at SW_80.2: now also D80.2 (A); no longer D80.1 (C)
- net at SW_81.2: now also D81.2 (A); no longer D81.1 (C)
- net at SW_82.2: now also D82.2 (A); no longer D82.1 (C)
- net at SW_83.2: now also D83.2 (A); no longer D83.1 (C)
- net at SW_84.2: now also D84.2 (A); no longer D84.1 (C)
- net at SW_85.2: now also D85.2 (A); no longer D85.1 (C)
- net at SW_86.2: now also D86.2 (A); no longer D86.1 (C)
- net at SW_87.2: now also D87.2 (A); no longer D87.1 (C)
- net at SW_88.2: now also D88.2 (A); no longer D88.1 (C)
- net at SW_89.2: now also D89.2 (A); no longer D89.1 (C)
- net at SW_90.2: now also D90.2 (A); no longer D90.1 (C)
- net at SW_91.2: now also D91.2 (A); no longer D91.1 (C)
- net at SW_92.2: now also D92.2 (A); no longer D92.1 (C)
- net at SW_93.2: now also D93.2 (A); no longer D93.1 (C)
- net at SW_94.2: now also D94.2 (A); no longer D94.1 (C)
- net at SW_95.2: now also D95.2 (A); no longer D95.1 (C)
- net at SW_96.2: now also D96.2 (A); no longer D96.1 (C)
- net at SW_97.2: now also D97.2 (A); no longer D97.1 (C)
- net at SW_98.2: now also D98.2 (A); no longer D98.1 (C)
- net at SW_99.2: now also D99.2 (A); no longer D99.1 (C)
- net at SW_100.2: now also D100.2 (A); no longer D100.1 (C)
- net at SW_101.2: now also D101.2 (A); no longer D101.1 (C)
- net at SW_102.2: now also D102.2 (A); no longer D102.1 (C)
- net at SW_103.2: now also D103.2 (A); no longer D103.1 (C)
- net at SW_104.2: now also D104.2 (A); no longer D104.1 (C)
- net at SW_105.2: now also D105.2 (A); no longer D105.1 (C)
- net at SW_106.2: now also D106.2 (A); no longer D106.1 (C)
- net at SW_107.2: now also D107.2 (A); no longer D107.1 (C)
- net at SW_108.2: now also D108.2 (A); no longer D108.1 (C)
- net at SW_109.2: now also D109.2 (A); no longer D109.1 (C)
- net at SW_110.2: now also D110.2 (A); no longer D110.1 (C)
- net at SW_111.2: now also D111.2 (A); no longer D111.1 (C)
- net at SW_112.2: now also D112.2 (A); no longer D112.1 (C)
- net at SW_113.2: now also D113.2 (A); no longer D113.1 (C)
- net at SW_114.2: now also D114.2 (A); no longer D114.1 (C)
- net at SW_115.2: now also D115.2 (A); no longer D115.1 (C)
- net at SW_116.2: now also D116.2 (A); no longer D116.1 (C)
- net at SW_117.2: now also D117.2 (A); no longer D117.1 (C)
- net at SW_118.2: now also D118.2 (A); no longer D118.1 (C)
- net at SW_119.2: now also D119.2 (A); no longer D119.1 (C)
- net at SW_120.2: now also D120.2 (A); no longer D120.1 (C)
- net at SW_121.2: now also D121.2 (A); no longer D121.1 (C)
- net at SW_122.2: now also D122.2 (A); no longer D122.1 (C)
- net at SW_123.2: now also D123.2 (A); no longer D123.1 (C)
- net at SW_124.2: now also D124.2 (A); no longer D124.1 (C)
- net at SW_125.2: now also D125.2 (A); no longer D125.1 (C)
- net at SW_126.2: now also D126.2 (A); no longer D126.1 (C)
- net at SW_127.2: now also D127.2 (A); no longer D127.1 (C)
- net at SW_128.2: now also D128.2 (A); no longer D128.1 (C)
- net at SW_129.2: now also D129.2 (A); no longer D129.1 (C)
- net at SW_130.2: now also D130.2 (A); no longer D130.1 (C)
- net at SW_131.2: now also D131.2 (A); no longer D131.1 (C)
- net at SW_132.2: now also D132.2 (A); no longer D132.1 (C)
- net at SW_133.2: now also D133.2 (A); no longer D133.1 (C)
- net at SW_134.2: now also D134.2 (A); no longer D134.1 (C)
- net at SW_135.2: now also D135.2 (A); no longer D135.1 (C)
- net at SW_136.2: now also D136.2 (A); no longer D136.1 (C)
- net at SW_137.2: now also D137.2 (A); no longer D137.1 (C)
- net at SW_138.2: now also D138.2 (A); no longer D138.1 (C)
- net at SW_139.2: now also D139.2 (A); no longer D139.1 (C)
- net at SW_140.2: now also D140.2 (A); no longer D140.1 (C)
- net at SW_141.2: now also D141.2 (A); no longer D141.1 (C)
- net at SW_142.2: now also D142.2 (A); no longer D142.1 (C)
- net at SW_143.2: now also D143.2 (A); no longer D143.1 (C)
- net at SW_144.2: now also D144.2 (A); no longer D144.1 (C)
- net at SW_145.2: now also D145.2 (A); no longer D145.1 (C)
- net at SW_146.2: now also D146.2 (A); no longer D146.1 (C)
- net at SW_147.2: now also D147.2 (A); no longer D147.1 (C)
- net at SW_148.2: now also D148.2 (A); no longer D148.1 (C)
- net at SW_149.2: now also D149.2 (A); no longer D149.1 (C)
- net at SW_150.2: now also D150.2 (A); no longer D150.1 (C)
- net at SW_151.2: now also D151.2 (A); no longer D151.1 (C)
- net at SW_152.2: now also D152.2 (A); no longer D152.1 (C)
- net at SW_153.2: now also D153.2 (A); no longer D153.1 (C)
- net at SW_154.2: now also D154.2 (A); no longer D154.1 (C)
- net at SW_155.2: now also D155.2 (A); no longer D155.1 (C)
- net at SW_156.2: now also D156.2 (A); no longer D156.1 (C)
- net at SW_157.2: now also D157.2 (A); no longer D157.1 (C)
- net at SW_158.2: now also D158.2 (A); no longer D158.1 (C)
- net at SW_159.2: now also D159.2 (A); no longer D159.1 (C)
- net at SW_160.2: now also D160.2 (A); no longer D160.1 (C)
- net at SW_161.2: now also D161.2 (A); no longer D161.1 (C)
- net at SW_162.2: now also D162.2 (A); no longer D162.1 (C)
- net at SW_163.2: now also D163.2 (A); no longer D163.1 (C)
- net at SW_164.2: now also D164.2 (A); no longer D164.1 (C)
- net at SW_165.2: now also D165.2 (A); no longer D165.1 (C)
- net at SW_166.2: now also D166.2 (A); no longer D166.1 (C)
- net at SW_167.2: now also D167.2 (A); no longer D167.1 (C)
- net at SW_168.2: now also D168.2 (A); no longer D168.1 (C)
- net at SW_169.2: now also D169.2 (A); no longer D169.1 (C)
- net at SW_170.2: now also D170.2 (A); no longer D170.1 (C)
- net at SW_171.2: now also D171.2 (A); no longer D171.1 (C)
- net at SW_172.2: now also D172.2 (A); no longer D172.1 (C)
- net at SW_173.2: now also D173.2 (A); no longer D173.1 (C)
- net at SW_174.2: now also D174.2 (A); no longer D174.1 (C)
- net at SW_175.2: now also D175.2 (A); no longer D175.1 (C)
- net at SW_176.2: now also D176.2 (A); no longer D176.1 (C)
- net at SW_177.2: now also D177.2 (A); no longer D177.1 (C)
- net at SW_178.2: now also D178.2 (A); no longer D178.1 (C)
- net at SW_179.2: now also D179.2 (A); no longer D179.1 (C)
- net at SW_180.2: now also D180.2 (A); no longer D180.1 (C)
- net at SW_181.2: now also D181.2 (A); no longer D181.1 (C)
- net at SW_182.2: now also D182.2 (A); no longer D182.1 (C)
- net at SW_183.2: now also D183.2 (A); no longer D183.1 (C)
- net at SW_184.2: now also D184.2 (A); no longer D184.1 (C)
- net at SW_185.2: now also D185.2 (A); no longer D185.1 (C)
- net at SW_186.2: now also D186.2 (A); no longer D186.1 (C)
- net at SW_187.2: now also D187.2 (A); no longer D187.1 (C)
- net at SW_188.2: now also D188.2 (A); no longer D188.1 (C)
- net at SW_189.2: now also D189.2 (A); no longer D189.1 (C)
- net at SW_190.2: now also D190.2 (A); no longer D190.1 (C)
- net at SW_191.2: now also D191.2 (A); no longer D191.1 (C)
- net at SW_192.2: now also D192.2 (A); no longer D192.1 (C)
- net at SW_193.2: now also D193.2 (A); no longer D193.1 (C)
- net at SW_194.2: now also D194.2 (A); no longer D194.1 (C)
- net at SW_195.2: now also D195.2 (A); no longer D195.1 (C)
- net at SW_196.2: now also D196.2 (A); no longer D196.1 (C)
- net at SW_197.2: now also D197.2 (A); no longer D197.1 (C)
- net at SW_198.2: now also D198.2 (A); no longer D198.1 (C)
- net at SW_199.2: now also D199.2 (A); no longer D199.1 (C)
- net at SW_200.2: now also D200.2 (A); no longer D200.1 (C)
- net at SW_201.2: now also D201.2 (A); no longer D201.1 (C)
- net at SW_202.2: now also D202.2 (A); no longer D202.1 (C)
- net at SW_203.2: now also D203.2 (A); no longer D203.1 (C)
- net at SW_204.2: now also D204.2 (A); no longer D204.1 (C)
- net at SW_205.2: now also D205.2 (A); no longer D205.1 (C)
- net at SW_206.2: now also D206.2 (A); no longer D206.1 (C)
- net at SW_207.2: now also D207.2 (A); no longer D207.1 (C)
- net at SW_208.2: now also D208.2 (A); no longer D208.1 (C)
- net at SW_209.2: now also D209.2 (A); no longer D209.1 (C)
- net at SW_210.2: now also D210.2 (A); no longer D210.1 (C)
- net at SW_211.2: now also D211.2 (A); no longer D211.1 (C)
- net at SW_212.2: now also D212.2 (A); no longer D212.1 (C)
- net at SW_213.2: now also D213.2 (A); no longer D213.1 (C)
- net at SW_214.2: now also D214.2 (A); no longer D214.1 (C)
- net at SW_215.2: now also D215.2 (A); no longer D215.1 (C)
- net at SW_216.2: now also D216.2 (A); no longer D216.1 (C)
- net at SW_217.2: now also D217.2 (A); no longer D217.1 (C)
- net at SW_218.2: now also D218.2 (A); no longer D218.1 (C)
- net at SW_219.2: now also D219.2 (A); no longer D219.1 (C)
- net at SW_220.2: now also D220.2 (A); no longer D220.1 (C)
- net at SW_221.2: now also D221.2 (A); no longer D221.1 (C)
- net at SW_222.2: now also D222.2 (A); no longer D222.1 (C)
- net at SW_223.2: now also D223.2 (A); no longer D223.1 (C)
- net at SW_224.2: now also D224.2 (A); no longer D224.1 (C)
- net at SW_225.2: now also D225.2 (A); no longer D225.1 (C)
